File: 2-Design/PCB/Four_Quad_DC_Motor_Drive/Converters.kicad_sch (KiCad schematic)
At the start: 12 parts, among them U6 ROE-0512S, U7 ROE-0512S, U8 SQL50

Commit message: Random Checkpoint
Changed lines of the file:
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@@
     (stroke (width 0) (type default) (color 0 0 0 0))
   )
-  (polyline (pts (xy 157.48 180.34) (xy 38.1 180.34))
+  (polyline (pts (xy 147.32 180.34) (xy 38.1 180.34))
     (stroke (width 0.254) (type solid) (color 132 0 0 1))
   )
@@
     (stroke (width 0) (type default) (color 0 0 0 0))
   )
-  (polyline (pts (xy 157.48 78.74) (xy 157.48 180.34))
+  (polyline (pts (xy 147.32 78.74) (xy 147.32 180.34))
     (stroke (width 0.254) (type solid) (color 132 0 0 1))
   )
@@
     (stroke (width 0) (type default) (color 0 0 0 0))
   )
-  (polyline (pts (xy 38.1 78.74) (xy 157.48 78.74))
+  (polyline (pts (xy 38.1 78.74) (xy 147.32 78.74))
     (stroke (width 0.254) (type solid) (color 132 0 0 1))
   )
